File: turbidity_sensor_module.sch (EAGLE design)
At the start: 29 parts, among them IC1 LTC485S, IC2 TINY441

Commit message: finishing touches, layed out pcb
Parts:
- removed JP3, JP4, JP5, JP6: (no value), sparkfun:M02PTH3
- removed R4, R5, R6: 4.7k, adafruit:R-US_R1206
- added D1: BP104GENERIC, opto-trans-siemens:BP104GENERIC
- added LED1, LED2, LED3: (no value), adafruit:LED5MM
- C2: value 1nF -> (none)
- R3: value 4.7k -> (none)
Connections:
- removed net A0: IC2.XTAL1/ADC11/PB0
- removed net A1: R6.1
- removed net A2: R5.1
- removed net A3: R4.1
- removed net THERM: C2.1, IC2.MISO/ADC0/AREF/PA0, JP3.1, R3.1
- net +5V: now also C2.1, D1.C, R3.1; no longer JP6.1, R3.2
- net GND: no longer JP3.2
- net MISO: no longer R5.2
- net MOSI: no longer R6.2
- net N$3: now also LED1.A, R10.2; no longer JP4.2, Q2.D
- net N$4: now also LED2.A, R11.2; no longer JP5.2, Q1.D
- net N$5: now also LED1.C, LED3.C, Q1.D; no longer JP5.1, R10.2
- net N$6: now also LED2.C, Q2.D; no longer JP4.1, R11.2
- net N$7: now also LED3.A, R3.2; no longer JP6.2, R12.1
- net PHOTODIODE: now also D1.A, R12.1
- net SCK: no longer R4.2
Other:
- moved on the sheet: C1, C2, C3, C4, C5, C6, IC1, IC2, ISP1, JP1, JP2, Q1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
