File: prototypes/rev1/optical_sensor_prototype.brd (EAGLE design)
At the start: 24.1 x 47.3 mm, 18 parts, among them IC1 QUAD_OPAMPD, IC2 LM50

Commit message: added remaining component values
Parts:
- R1: value (none) -> 24.3
- R2, R3, R4, R5: value (none) -> 10k
Changed lines of the file:
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@@
 <attribute name="NAME" x="2.8575" y="9.652" size="1.27" layer="25" font="vector"/>
 </element>
-<element name="R1" library="adafruit" package="R1206" value="" x="-8.89" y="21.59" smashed="yes">
+<element name="R1" library="adafruit" package="R1206" value="24.3" x="-8.89" y="21.59" smashed="yes">
 <attribute name="NAME" x="-6.1595" y="21.7805" size="1.27" layer="25" font="vector"/>
 <attribute name="VALUE" x="-10.287" y="19.177" size="1.27" layer="27"/>
 </element>
-<element name="R2" library="adafruit" package="R1206" value="" x="8.89" y="19.05" smashed="yes" rot="R270">
+<element name="R2" library="adafruit" package="R1206" value="10k" x="8.89" y="19.05" smashed="yes" rot="R270">
 <attribute name="NAME" x="10.3505" y="20.1295" size="1.27" layer="25" font="vector" rot="R270"/>
 <attribute name="VALUE" x="6.477" y="20.447" size="1.27" layer="27" rot="R270"/>
 </element>
-<element name="R3" library="adafruit" package="R1206" value="" x="8.89" y="12.7" smashed="yes" rot="R90">
+<element name="R3" library="adafruit" package="R1206" value="10k" x="8.89" y="12.7" smashed="yes" rot="R90">
 <attribute name="NAME" x="11.557" y="11.6205" size="1.27" layer="25" font="vector" rot="R90"/>
 <attribute name="VALUE" x="11.303" y="11.303" size="1.27" layer="27" rot="R90"/>
 </element>
-<element name="R4" library="adafruit" package="R1206" value="" x="-3.81" y="12.7" smashed="yes" rot="R90">
+<element name="R4" library="adafruit" package="R1206" value="10k" x="-3.81" y="12.7" smashed="yes" rot="R90">
 <attribute name="NAME" x="-5.2705" y="11.303" size="1.27" layer="25" font="vector" rot="R90"/>
 <attribute name="VALUE" x="-1.397" y="11.303" size="1.27" layer="27" rot="R90"/>
 </element>
-<element name="R5" library="adafruit" package="R1206" value="" x="-3.81" y="19.05" smashed="yes" rot="R270">
+<element name="R5" library="adafruit" package="R1206" value="10k" x="-3.81" y="19.05" smashed="yes" rot="R270">
 <attribute name="NAME" x="-2.3495" y="20.447" size="1.27" layer="25" font="vector" rot="R270"/>
 <attribute name="VALUE" x="-6.223" y="20.447" size="1.27" layer="27" rot="R270"/>
